File: src/server/schematicToTyped/fixtures/led_smd.sch (EAGLE design)
At the start: 2 parts

Commit message: Improve fixtures
Connections:
- net <GPIO renamed #GPIO_3.3V
Changed lines of the file:
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@@
 </segment>
 </net>
-<net name="&lt;GPIO" class="0">
+<net name="#GPIO_3.3V" class="0">
 <segment>
 <pinref part="D1" gate="G$1" pin="A"/>
