File: server/data/typedSchematics/atmega328.brd (EAGLE design)
At the start: 15.4 x 31.1 mm, 7 parts, among them U3 ATMEGA328, Y1 8MHz

Commit message: Redefining typed annotation
Connections:
- net !#ADC0 renamed #ADC-0
- net #ADC1 renamed #ADC-1
- net #ADC2 renamed #ADC-2
- net #ADC3 renamed #ADC-3
- net #ADC6 renamed #ADC-6
- net #ADC7 renamed #ADC-7
- net #AIN0||#GPIO6 renamed #AIN-0||#GPIO-6
- net #AIN1||#GPIO7 renamed #AIN-1||#GPIO-7
- net #GPIO10 renamed #GPIO-10
- net #GPIO9 renamed #GPIO-9
- net #I2C0.SCL||#ADC5 renamed #I2C-0.SCL||#ADC-5
- net #I2C0.SDA||#ADC4 renamed #I2C-0.SDA||#ADC-4
- net #ICP0||#GPIO8 renamed #ICP-0||#GPIO-8
- net #INT0||#GPIO2 renamed #INT-0||#GPIO-2
- net #INT1||#GPIO3 renamed #INT-1||#GPIO-3
- net #SERIAL0.RX||#GPIO0 renamed #SERIAL-0.RX||#GPIO-0
- net #SERIAL0.TX||#GPIO1 renamed #SERIAL-0.TX||#GPIO-1
- net #SPI0.MISO||#GPIO12 renamed #SPI-0.MISO||#GPIO-12
- net #SPI0.MOSI||#GPIO11 renamed #SPI-0.MOSI||#GPIO-11
- net #SPI0.SCK||#GPIO13 renamed #SPI-0.SCK||#GPIO-13
- net #T0||#GPIO4 renamed #T-0||#GPIO-4
- net #T1||#GPIO5 renamed #T-1||#GPIO-5
Changed lines of the file:
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@@
 <contactref element="C3" pad="1"/>
 </signal>
-<signal name="!#ADC0">
+<signal name="#ADC-0">
 <contactref element="U3" pad="23"/>
 </signal>
-<signal name="#ADC1">
+<signal name="#ADC-1">
 <contactref element="U3" pad="24"/>
 </signal>
-<signal name="#ADC2">
+<signal name="#ADC-2">
 <contactref element="U3" pad="25"/>
 </signal>
-<signal name="#ADC3">
+<signal name="#ADC-3">
 <contactref element="U3" pad="26"/>
 </signal>
-<signal name="#I2C0.SDA||#ADC4">
+<signal name="#I2C-0.SDA||#ADC-4">
 <contactref element="U3" pad="27"/>
 </signal>
-<signal name="#I2C0.SCL||#ADC5">
+<signal name="#I2C-0.SCL||#ADC-5">
 <contactref element="U3" pad="28"/>
 </signal>
-<signal name="#ADC6">
+<signal name="#ADC-6">
 <contactref element="U3" pad="19"/>
 </signal>
-<signal name="#ADC7">
+<signal name="#ADC-7">
 <contactref element="U3" pad="22"/>
 </signal>
-<signal name="#SPI0.MOSI||#GPIO11">
+<signal name="#SPI-0.MOSI||#GPIO-11">
 <contactref element="JP4" pad="4"/>
 <contactref element="U3" pad="15"/>
@@
 <wire x1="4.8768" y1="2.0574" x2="4.84" y2="2.05" width="0.1524" layer="1"/>
 </signal>
-<signal name="#SPI0.MISO||#GPIO12">
+<signal name="#SPI-0.MISO||#GPIO-12">
 <contactref element="U3" pad="16"/>
 <contactref element="JP4" pad="1"/>
@@
 <wire x1="7.3914" y1="4.6482" x2="7.38" y2="4.59" width="0.1524" layer="1"/>
 </signal>
-<signal name="#SPI0.SCK||#GPIO13">
+<signal name="#SPI-0.SCK||#GPIO-13">
 <contactref element="JP4" pad="3"/>
 <contactref element="U3" pad="17"/>
@@
 <wire x1="4.8768" y1="4.6482" x2="4.84" y2="4.59" width="0.1524" layer="1"/>
 </signal>
-<signal name="#SERIAL0.RX||#GPIO0">
+<signal name="#SERIAL-0.RX||#GPIO-0">
 <contactref element="U3" pad="30"/>
 </signal>
-<signal name="#SERIAL0.TX||#GPIO1">
+<signal name="#SERIAL-0.TX||#GPIO-1">
 <contactref element="U3" pad="31"/>
 </signal>
-<signal name="#INT0||#GPIO2">
+<signal name="#INT-0||#GPIO-2">
 <contactref element="U3" pad="32"/>
 </signal>
-<signal name="#INT1||#GPIO3">
+<signal name="#INT-1||#GPIO-3">
 <contactref element="U3" pad="1"/>
 </signal>
-<signal name="#T0||#GPIO4">
+<signal name="#T-0||#GPIO-4">
 <contactref element="U3" pad="2"/>
 </signal>
-<signal name="#T1||#GPIO5">
+<signal name="#T-1||#GPIO-5">
 <contactref element="U3" pad="9"/>
 </signal>
-<signal name="#AIN0||#GPIO6">
+<signal name="#AIN-0||#GPIO-6">
 <contactref element="U3" pad="10"/>
 </signal>
-<signal name="#AIN1||#GPIO7">
+<signal name="#AIN-1||#GPIO-7">
 <contactref element="U3" pad="11"/>
 </signal>
-<signal name="#ICP0||#GPIO8">
+<signal name="#ICP-0||#GPIO-8">
 <contactref element="U3" pad="12"/>
 </signal>
-<signal name="#GPIO9">
+<signal name="#GPIO-9">
 <contactref element="U3" pad="13"/>
 </signal>
-<signal name="#GPIO10">
+<signal name="#GPIO-10">
 <contactref element="U3" pad="14"/>
 </signal>

Commit message: Add typed power
Connections:
- new net @VIN_5V: JP4.2, R4.2
- net VCC: no longer JP4.2, R4.2
Changed lines of the file:
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@@
 </signal>
 <signal name="VCC" class="1">
-<contactref element="R4" pad="2"/>
 <contactref element="U3" pad="4"/>
 <contactref element="U3" pad="6"/>
 <contactref element="U3" pad="18"/>
-<contactref element="JP4" pad="2"/>
 <wire x1="5.053" y1="14.197" x2="4.1148" y2="14.197" width="0.381" layer="1"/>
 <wire x1="4.1148" y1="14.1732" x2="1.9812" y2="14.1732" width="0.381" layer="1"/>
 <wire x1="5.1054" y1="14.2494" x2="5.053" y2="14.197" width="0.381" layer="1"/>
-<wire x1="1.9812" y1="14.1732" x2="1.93" y2="14.22" width="0.381" layer="1"/>
 <wire x1="5.1054" y1="14.2494" x2="5.1074" y2="14.27" width="0.381" layer="1"/>
 <wire x1="4.4196" y1="12.7254" x2="5.1054" y2="12.7254" width="0.381" layer="1"/>
@@
 <wire x1="8.6868" y1="4.0386" x2="7.3914" y2="2.7432" width="0.381" layer="16"/>
 <wire x1="8.6868" y1="11.7348" x2="8.6868" y2="4.0386" width="0.381" layer="16"/>
-<wire x1="7.3914" y1="2.0574" x2="7.38" y2="2.05" width="0.381" layer="16"/>
 <wire x1="8.6868" y1="11.7348" x2="8.6868" y2="11.8872" width="0.381" layer="1"/>
 <via x="8.6868" y="11.7348" extent="1-16" drill="0.35"/>
@@
 <contactref element="U3" pad="14"/>
 </signal>
+<signal name="@VIN_5V">
+<contactref element="R4" pad="2"/>
+<contactref element="JP4" pad="2"/>
+<wire x1="7.38" y1="2.05" x2="1.93" y2="14.22" width="0" layer="19" extent="1-1"/>
+</signal>
 </signals>

Commit message: Adding I2C options in schematic + Voltage fix
Connections:
- net @VIN_5V renamed @VIN_3.3V-5V
Changed lines of the file:
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@@
 <contactref element="U3" pad="14"/>
 </signal>
-<signal name="@VIN_5V">
+<signal name="@VIN_3.3V-5V">
 <contactref element="R4" pad="2"/>
 <contactref element="JP4" pad="2"/>

Commit message: Adding required annotation symbol
Connections:
- net #ADC-0 renamed #ADC-0!
- net #ADC-1 renamed #ADC-1!
- net #ADC-2 renamed #ADC-2!
- net #ADC-3 renamed #ADC-3!
- net #ADC-6 renamed #ADC-6!
- net #ADC-7 renamed #ADC-7!
- net #AIN-0||#GPIO-6 renamed #AIN-0!||#GPIO-6!
- net #AIN-1||#GPIO-7 renamed #AIN-1!||#GPIO-7!
- net #GPIO-10 renamed #GPIO-10!
- net #GPIO-9 renamed #GPIO-9!
- net #GPIO-DTR renamed #GPIO-DTR!
- net #GPIO-RESET renamed #GPIO-RESET!
- net #I2C-0.SCL||#ADC-5 renamed #I2C-0.SCL!||#ADC-5!
- net #I2C-0.SDA||#ADC-4 renamed #I2C-0.SDA!||#ADC-4!
- net #ICP-0||#GPIO-8 renamed #GPIO-8!
- net #INT-0||#GPIO-2 renamed #GPIO-2!
- net #INT-1||#GPIO-3 renamed #GPIO-3!
- net #SERIAL-0.RX||#GPIO-0 renamed #SERIAL-0.RX!||#GPIO-0!
- net #SERIAL-0.TX||#GPIO-1 renamed #SERIAL-0.TX!||#GPIO-1!
- net #SPI-0.MISO||#GPIO-12 renamed #SPI-0.MISO!||#GPIO-12!
- net #SPI-0.MOSI||#GPIO-11 renamed #SPI-0.MOSI!||#GPIO-11!
- net #SPI-0.SCK||#GPIO-13 renamed #SPI-0.SCK!||#GPIO-13!
- net #T-0||#GPIO-4 renamed #GPIO-4!
- net #T-1||#GPIO-5 renamed #GPIO-5!
Changed lines of the file:
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@@
 <via x="8.6868" y="11.7348" extent="1-16" drill="0.35"/>
 </signal>
-<signal name="#GPIO-RESET">
+<signal name="#GPIO-RESET!">
 <contactref element="U3" pad="29"/>
 <contactref element="R4" pad="1"/>
@@
 <via x="12.4968" y="14.0208" extent="1-16" drill="0.35"/>
 </signal>
-<signal name="#GPIO-DTR">
+<signal name="#GPIO-DTR!">
 <contactref element="C3" pad="1"/>
 </signal>
-<signal name="#ADC-0">
+<signal name="#ADC-0!">
 <contactref element="U3" pad="23"/>
 </signal>
-<signal name="#ADC-1">
+<signal name="#ADC-1!">
 <contactref element="U3" pad="24"/>
 </signal>
-<signal name="#ADC-2">
+<signal name="#ADC-2!">
 <contactref element="U3" pad="25"/>
 </signal>
-<signal name="#ADC-3">
+<signal name="#ADC-3!">
 <contactref element="U3" pad="26"/>
 </signal>
-<signal name="#I2C-0.SDA||#ADC-4">
+<signal name="#I2C-0.SDA!||#ADC-4!">
 <contactref element="U3" pad="27"/>
 </signal>
-<signal name="#I2C-0.SCL||#ADC-5">
+<signal name="#I2C-0.SCL!||#ADC-5!">
 <contactref element="U3" pad="28"/>
 </signal>
-<signal name="#ADC-6">
+<signal name="#ADC-6!">
 <contactref element="U3" pad="19"/>
 </signal>
-<signal name="#ADC-7">
+<signal name="#ADC-7!">
 <contactref element="U3" pad="22"/>
 </signal>
-<signal name="#SPI-0.MOSI||#GPIO-11">
+<signal name="#SPI-0.MOSI!||#GPIO-11!">
 <contactref element="JP4" pad="4"/>
 <contactref element="U3" pad="15"/>
@@
 <wire x1="4.8768" y1="2.0574" x2="4.84" y2="2.05" width="0.1524" layer="1"/>
 </signal>
-<signal name="#SPI-0.MISO||#GPIO-12">
+<signal name="#SPI-0.MISO!||#GPIO-12!">
 <contactref element="U3" pad="16"/>
 <contactref element="JP4" pad="1"/>
@@
 <wire x1="7.3914" y1="4.6482" x2="7.38" y2="4.59" width="0.1524" layer="1"/>
 </signal>
-<signal name="#SPI-0.SCK||#GPIO-13">
+<signal name="#SPI-0.SCK!||#GPIO-13!">
 <contactref element="JP4" pad="3"/>
 <contactref element="U3" pad="17"/>
@@
 <wire x1="4.8768" y1="4.6482" x2="4.84" y2="4.59" width="0.1524" layer="1"/>
 </signal>
-<signal name="#SERIAL-0.RX||#GPIO-0">
+<signal name="#SERIAL-0.RX!||#GPIO-0!">
 <contactref element="U3" pad="30"/>
 </signal>
-<signal name="#SERIAL-0.TX||#GPIO-1">
+<signal name="#SERIAL-0.TX!||#GPIO-1!">
 <contactref element="U3" pad="31"/>
 </signal>
-<signal name="#INT-0||#GPIO-2">
+<signal name="#GPIO-2!">
 <contactref element="U3" pad="32"/>
 </signal>
-<signal name="#INT-1||#GPIO-3">
+<signal name="#GPIO-3!">
 <contactref element="U3" pad="1"/>
 </signal>
-<signal name="#T-0||#GPIO-4">
+<signal name="#GPIO-4!">
 <contactref element="U3" pad="2"/>
 </signal>
-<signal name="#T-1||#GPIO-5">
+<signal name="#GPIO-5!">
 <contactref element="U3" pad="9"/>
 </signal>
-<signal name="#AIN-0||#GPIO-6">
+<signal name="#AIN-0!||#GPIO-6!">
 <contactref element="U3" pad="10"/>
 </signal>
-<signal name="#AIN-1||#GPIO-7">
+<signal name="#AIN-1!||#GPIO-7!">
 <contactref element="U3" pad="11"/>
 </signal>
-<signal name="#ICP-0||#GPIO-8">
+<signal name="#GPIO-8!">
 <contactref element="U3" pad="12"/>
 </signal>
-<signal name="#GPIO-9">
+<signal name="#GPIO-9!">
 <contactref element="U3" pad="13"/>
 </signal>
-<signal name="#GPIO-10">
+<signal name="#GPIO-10!">
 <contactref element="U3" pad="14"/>
 </signal>
