File: server/data/typedSchematics/flash.sch (EAGLE design)
At the start: 2 parts, among them IC1 M25P80VMN6TPBA

Commit message: Adding master-slave constrain to SPI
Other:
- note added: "#{ SPI:{arch:slave} }"
Changed lines of the file:
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@@
 <plain>
 <text x="30.48" y="7.62" size="2.54" layer="97">FLASH</text>
+<text x="83.82" y="25.4" size="1.778" layer="97">#{
+SPI:{arch:slave}
+}</text>
 </plain>
 <instances>
@@
 </drawing>
 <compatibility>
+<note version="6.3" minversion="6.2.2" severity="warning">
+Since Version 6.2.2 text objects can contain more than one line,
+which will not be processed correctly with this version.
+</note>
 <note version="8.2" severity="warning">
 Since Version 8.2, EAGLE supports online libraries. The ids

Commit message: Add typed power
Connections:
- net VDD renamed @VIN_5V
Changed lines of the file:
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@@
 <part name="IC1" library="M25P80VMN6TPBA" deviceset="M25P80VMN6TPBA" device=""/>
 <part name="C1" library="SparkFun-Capacitors" library_urn="urn:adsk.eagle:library:510" deviceset="0.1UF" device="-0603-25V-(+80/-20%)" package3d_urn="urn:adsk.eagle:package:37414/1" value="0.1uF"/>
-<part name="SUPPLY1" library="SparkFun-PowerSymbols" library_urn="urn:adsk.eagle:library:530" deviceset="VDD" device=""/>
 <part name="GND1" library="SparkFun-PowerSymbols" library_urn="urn:adsk.eagle:library:530" deviceset="GND" device=""/>
 <part name="GND2" library="SparkFun-PowerSymbols" library_urn="urn:adsk.eagle:library:530" deviceset="GND" device=""/>
@@
 <attribute name="VALUE" x="75.184" y="15.621" size="1.778" layer="96" font="vector"/>
 </instance>
-<instance part="SUPPLY1" gate="VDD" x="73.66" y="33.02" smashed="yes">
-<attribute name="VALUE" x="73.66" y="35.814" size="1.778" layer="96" align="bottom-center"/>
-</instance>
 <instance part="GND1" gate="1" x="73.66" y="7.62" smashed="yes">
 <attribute name="VALUE" x="73.66" y="7.366" size="1.778" layer="96" align="top-center"/>
@@
 </busses>
 <nets>
-<net name="VDD" class="0">
-<segment>
-<pinref part="SUPPLY1" gate="VDD" pin="VDD"/>
-<pinref part="C1" gate="G$1" pin="1"/>
-<wire x1="73.66" y1="33.02" x2="73.66" y2="27.94" width="0.1524" layer="91"/>
-<pinref part="IC1" gate="G$1" pin="VCC"/>
-<wire x1="73.66" y1="27.94" x2="73.66" y2="22.86" width="0.1524" layer="91"/>
-<wire x1="50.8" y1="22.86" x2="53.34" y2="22.86" width="0.1524" layer="91"/>
-<wire x1="53.34" y1="22.86" x2="53.34" y2="27.94" width="0.1524" layer="91"/>
-<wire x1="53.34" y1="27.94" x2="73.66" y2="27.94" width="0.1524" layer="91"/>
-<junction x="73.66" y="27.94"/>
-</segment>
-</net>
 <net name="GND" class="0">
 <segment>
@@
 </segment>
 </net>
+<net name="@VIN_5V" class="0">
+<segment>
+<pinref part="C1" gate="G$1" pin="1"/>
+<pinref part="IC1" gate="G$1" pin="VCC"/>
+<wire x1="73.66" y1="27.94" x2="73.66" y2="22.86" width="0.1524" layer="91"/>
+<wire x1="50.8" y1="22.86" x2="53.34" y2="22.86" width="0.1524" layer="91"/>
+<wire x1="53.34" y1="22.86" x2="53.34" y2="27.94" width="0.1524" layer="91"/>
+<wire x1="53.34" y1="27.94" x2="73.66" y2="27.94" width="0.1524" layer="91"/>
+<wire x1="73.66" y1="27.94" x2="73.66" y2="35.56" width="0.1524" layer="91"/>
+<junction x="73.66" y="27.94"/>
+<wire x1="73.66" y1="35.56" x2="68.58" y2="35.56" width="0.1524" layer="91"/>
+<label x="68.58" y="35.56" size="1.27" layer="95" rot="R180" xref="yes"/>
+</segment>
+</net>

Commit message: Schematics with require annotation
Connections:
- net #GPIO-HOLD renamed #GPIO-HOLD!
- net #GPIO-WP renamed #GPIO-WP!
Changed lines of the file:
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@@
 </segment>
 </net>
-<net name="#GPIO-HOLD" class="0">
+<net name="#GPIO-HOLD!" class="0">
 <segment>
 <pinref part="IC1" gate="G$1" pin="HOLD#"/>
@@
 </segment>
 </net>
-<net name="#GPIO-WP" class="0">
+<net name="#GPIO-WP!" class="0">
 <segment>
 <pinref part="IC1" gate="G$1" pin="W#"/>
