File: client/public/data/typedSchematics/atmega328.brd (EAGLE design)
At the start: 15.4 x 31.1 mm, 7 parts, among them U3 ATMEGA328, Y1 8MHz

Commit message: Configuring schematics with blocktype info
Connections:
- net #AIN-0!||#GPIO-6! renamed #GPIO-6!||#AIN-0!
- net #AIN-1!||#GPIO-7! renamed #GPIO-7!||#AIN-1!
Changed lines of the file:
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@@
 <contactref element="U3" pad="9"/>
 </signal>
-<signal name="#AIN-0!||#GPIO-6!">
+<signal name="#GPIO-6!||#AIN-0!">
 <contactref element="U3" pad="10"/>
 </signal>
-<signal name="#AIN-1!||#GPIO-7!">
+<signal name="#GPIO-7!||#AIN-1!">
 <contactref element="U3" pad="11"/>
 </signal>
