File: client/public/data/typedSchematics/temperature_sensor.sch (EAGLE design)
At the start: 1 part, among them U1 MCP9808

Commit message: Configuring schematics with blocktype info
Other:
- note added: "#{ BlockType:Pheripherial, I2C:{arch:slave,address:'0x18'}, }"
- note removed: "#{ I2C:{arch:slave,address:'0x18'}, }"
Changed lines of the file:
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@@
 <plain>
 <text x="22.86" y="-2.54" size="1.778" layer="97">#{
+BlockType:Pheripherial,
 I2C:{arch:slave,address:'0x18'},
 }</text>
