File: client/public/data/typedSchematics/led_smd.brd (EAGLE design)
At the start: 6.5 x 6.6 mm, 2 parts

Commit message: Adding GPIO altname for led typed schematic
Connections:
- net #GPIO renamed #GPIO-0
Changed lines of the file:
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@@
 <wire x1="2.04" y1="1.91" x2="4.68" y2="1.91" width="0.508" layer="1"/>
 </signal>
-<signal name="#GPIO">
+<signal name="#GPIO-0">
 <contactref element="D1" pad="A"/>
 </signal>
