File: server/scripts/mergeOutput/merged.sch (EAGLE design)
At the start: 15 parts, among them IC1__u1 AMS1117-5.0, J1__u0 DCJ0202, U3__u2 ATMEGA328, Y1__u2 8MHz

Commit message: Cleaning server side
Parts:
- removed C3__u2, C6__u2: 0.1uF, SparkFun-Capacitors__u2:0.1UF-0603-25V-5%
- removed D1__u3: (no value), SparkFun-LED__u3:LED1206
- removed JP4__u2: AVR_SPI, SparkFun__u2:AVR_SPI_PRG_6PTH
- removed R1__u3: 330, SparkFun-Resistors__u3:RESISTOR1206
- removed R4__u2: 10k, SparkFun-Resistors__u2:10KOHM-0603-1/10W-1%
- removed S2__u2: MOMENTARY-SWITCH-SPST-SMD-6.2MM-TALL, SparkFun-Switches__u2:MOMENTARY-SWITCH-SPST-SMD-6.2MM-TALL
- removed U3__u2: ATMEGA328, SparkFun__u2:ATMEGA168
- removed Y1__u2: 8MHz, SparkFun__u2:RESONATORSMD
- added C1__u2: 0.1uF, SparkFun-Capacitors__u2:0.1UF-0603-25V-(+80/-20%)
- added C3__u3, C6__u3: 0.1uF, SparkFun-Capacitors__u3:0.1UF-0603-25V-5%
- added IC1__u2: M25P80VMN6TPBA, M25P80VMN6TPBA__u2:M25P80VMN6TPBA
- added JP4__u3: AVR_SPI, SparkFun__u3:AVR_SPI_PRG_6PTH
- added R4__u3: 10k, SparkFun-Resistors__u3:10KOHM-0603-1/10W-1%
- added S2__u3: MOMENTARY-SWITCH-SPST-SMD-6.2MM-TALL, SparkFun-Switches__u3:MOMENTARY-SWITCH-SPST-SMD-6.2MM-TALL
- added U3__u3: ATMEGA328, SparkFun__u3:ATMEGA168
- added Y1__u3: 8MHz, SparkFun__u3:RESONATORSMD
Connections:
- removed net #ADC-0!__u2: U3__u2.PC0(ADC0)
- removed net #ADC-1!__u2: U3__u2.PC1(ADC1)
- removed net #ADC-2!__u2: U3__u2.PC2(ADC2)
- removed net #ADC-3!__u2: U3__u2.PC3(ADC3)
- removed net #ADC-6!__u2: U3__u2.ADC6
- removed net #ADC-7!__u2: U3__u2.ADC7
- removed net #GPIO-10!__u2: U3__u2.PB2(SS/OC1B)
- removed net #GPIO-2!+#GPIO: D1__u3.A, U3__u2.PD2(INT0)
- removed net #GPIO-3!__u2: U3__u2.PD3(INT1)
- removed net #GPIO-4!__u2: U3__u2.PD4(XCK/T0)
- removed net #GPIO-5!__u2: U3__u2.PD5(T1)
- removed net #GPIO-6!||#AIN-0!__u2: U3__u2.PD6(AIN0)
- removed net #GPIO-7!||#AIN-1!__u2: U3__u2.PD7(AIN1)
- removed net #GPIO-8!__u2: U3__u2.PB0(ICP)
- removed net #GPIO-9!__u2: U3__u2.PB1(OC1A)
- removed net #GPIO-DTR!__u2: C3__u2.1
- removed net #GPIO-RESET!__u2: C3__u2.2, JP4__u2.5, R4__u2.1, S2__u2.2, U3__u2.PC6(/RESET)
- removed net #I2C-0.SCL!||#ADC-5!__u2: U3__u2.PC5(ADC5/SCL)
- removed net #I2C-0.SDA!||#ADC-4!__u2: U3__u2.PC4(ADC4/SDA)
- removed net #SERIAL-0.RX!||#GPIO-0!__u2: U3__u2.PD0(RXD)
- removed net #SERIAL-0.TX!||#GPIO-1!__u2: U3__u2.PD1(TXD)
- removed net #SPI-0.MISO!||#GPIO-12!__u2: JP4__u2.1, U3__u2.PB4(MISO)
- removed net #SPI-0.MOSI!||#GPIO-11!__u2: JP4__u2.4, U3__u2.PB3(MOSI/OC2)
- removed net #SPI-0.SCK!||#GPIO-13!__u2: JP4__u2.3, U3__u2.PB5(SCK)
- removed net @VOUT_5V+@VIN_3.3V-5V: C1__u1.1, IC1__u1.TB, IC1__u1.VOUT, JP4__u2.2, R4__u2.2
- removed net AREF__u2: C6__u2.1, U3__u2.AREF
- removed net N$10__u2: U3__u2.PB6(XTAL1/TOSC1), Y1__u2.3
- removed net N$12__u2: U3__u2.PB7(XTAL2/TOSC2), Y1__u2.1
- removed net N$1__u3: D1__u3.C, R1__u3.2
- removed net VCC__u2: U3__u2.AVCC, U3__u2.VCC@1, U3__u2.VCC@2
- new net #ADC-0!__u3: U3__u3.PC0(ADC0)
- new net #ADC-1!__u3: U3__u3.PC1(ADC1)
- new net #ADC-2!__u3: U3__u3.PC2(ADC2)
- new net #ADC-3!__u3: U3__u3.PC3(ADC3)
- new net #ADC-6!__u3: U3__u3.ADC6
- new net #ADC-7!__u3: U3__u3.ADC7
- new net #GPIO-10!__u3: U3__u3.PB2(SS/OC1B)
- new net #GPIO-2!+#GPIO-WP!: IC1__u2.W#, U3__u3.PD2(INT0)
- new net #GPIO-3!+#GPIO-CS: IC1__u2.S#, U3__u3.PD3(INT1)
- new net #GPIO-4!+#GPIO-HOLD!: IC1__u2.HOLD#, U3__u3.PD4(XCK/T0)
- new net #GPIO-5!__u3: U3__u3.PD5(T1)
- new net #GPIO-6!||#AIN-0!__u3: U3__u3.PD6(AIN0)
- new net #GPIO-7!||#AIN-1!__u3: U3__u3.PD7(AIN1)
- new net #GPIO-8!__u3: U3__u3.PB0(ICP)
- new net #GPIO-9!__u3: U3__u3.PB1(OC1A)
- new net #GPIO-DTR!__u3: C3__u3.1
- new net #GPIO-RESET!__u3: C3__u3.2, JP4__u3.5, R4__u3.1, S2__u3.2, U3__u3.PC6(/RESET)
- new net #I2C-0.SCL!||#ADC-5!__u3: U3__u3.PC5(ADC5/SCL)
- new net #I2C-0.SDA!||#ADC-4!__u3: U3__u3.PC4(ADC4/SDA)
- new net #SERIAL-0.RX!||#GPIO-0!__u3: U3__u3.PD0(RXD)
- new net #SERIAL-0.TX!||#GPIO-1!__u3: U3__u3.PD1(TXD)
- new net #SPI-0.MISO!||#GPIO-12!+#SPI.MISO: IC1__u2.DQ1, JP4__u3.1, U3__u3.PB4(MISO)
- new net #SPI-0.MOSI!||#GPIO-11!+#SPI.MOSI: IC1__u2.DQ0, JP4__u3.4, U3__u3.PB3(MOSI/OC2)
- new net #SPI-0.SCK!||#GPIO-13!+#SPI.SCK: IC1__u2.C, JP4__u3.3, U3__u3.PB5(SCK)
- new net @VIN_3.3V-5V__u3: JP4__u3.2, R4__u3.2
- new net @VOUT_5V+@VIN_5V: C1__u1.1, C1__u2.1, IC1__u1.TB, IC1__u1.VOUT, IC1__u2.VCC
- new net AREF__u3: C6__u3.1, U3__u3.AREF
- new net N$10__u3: U3__u3.PB6(XTAL1/TOSC1), Y1__u3.3
- new net N$12__u3: U3__u3.PB7(XTAL2/TOSC2), Y1__u3.1
- new net VCC__u3: U3__u3.AVCC, U3__u3.VCC@1, U3__u3.VCC@2
- net GND: now also C1__u2.2, C6__u3.2, IC1__u2.VSS, JP4__u3.6, S2__u3.1, U3__u3.AGND, U3__u3.GND@1, U3__u3.GND@2, Y1__u3.2; no longer C6__u2.2, JP4__u2.6, R1__u3.1, S2__u2.1, U3__u2.AGND, U3__u2.GND@1, U3__u2.GND@2, Y1__u2.2
Other:
- note added: "#{ BlockType:Pheripherial, SPI:{arch:slave} }"
- note added: "FLASH"
- note removed: "#{ BlockType:Pheripherial, }"
